File: kicad/Performer-SE-PL-CL.kicad_pcb (KiCad board)
At the start: 4 copper layers, 125.7 x 109.2 mm, 42 parts, among them IC1 MC68000P, J1 MAC_SE_PDS, U1 MC68030RC, U2 MC68881FN-SOC, U3 ATF16V8BJ, U4 ATF16V8BJ, U5 ATF16V8BJ, U6 ATF16V8BJ, U7 ATF16V8BJ

Commit message: Rename MC68030 Kicad footprint
Parts:
- U1: footprint project:CPGA-169_68030 -> project:CPGA-169_MC68030
Changed lines of the file:
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@@
 		)
 	)
-	(footprint "project:CPGA-169_68030"
+	(footprint "project:CPGA-169_MC68030"
 		(layer "F.Cu")
 		(at 118.8898 59.2777 90)
@@
 			)
 		)
-		(property "Footprint" "project:CPGA-169_68030"
+		(property "Footprint" "project:CPGA-169_MC68030"
 			(at 0 0 0)
 			(unlocked yes)
@@
 			(pintype "bidirectional")
 		)
-		(model "${KICAD8_3DMODEL_DIR}/Package_BGA.3dshapes/Xilinx_CPGA196.wrl"
-			(offset
-				(xyz 0 0 0)
-			)
-			(scale
-				(xyz 1 1 1)
-			)
-			(rotate
-				(xyz 0 0 0)
-			)
-		)
 	)

Commit message: Update the MC68030 footprint
Parts:
- U1: footprint project:CPGA-169_MC68030 -> project:CPGA-128_Layout13x13_MC68030
Changed lines of the file:
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@@
 		)
 	)
-	(footprint "project:CPGA-169_MC68030"
+	(footprint "project:CPGA-128_Layout13x13_MC68030"
 		(layer "F.Cu")
 		(at 118.8898 59.2777 90)
 		(descr "MC68030, 13x13 Layout, 2.54mm Pitch")
-		(tags "CPGA-169 2.54 68030")
+		(tags "CPGA-128 2.54 68030")
 		(property "Reference" "U1"
 			(at -19.05 0 0)
@@
 			)
 		)
-		(property "Footprint" "project:CPGA-169_MC68030"
+		(property "Footprint" "project:CPGA-128_Layout13x13_MC68030"
 			(at 0 0 0)
 			(unlocked yes)

Commit message: Update PDS footprint of the Performer-SE-PL-CL
Parts:
- J1: footprint project:DIN41612_R_3x32_Male_Vertical_THT_Mirror -> project:DIN41612_R_3x32_Male_Vertical_THT_Mirror_NoMountingHoles
Changed lines of the file:
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@@
 		)
 	)
-	(footprint "project:DIN41612_R_3x32_Male_Vertical_THT_Mirror"
+	(footprint "project:DIN41612_R_3x32_Male_Vertical_THT_Mirror_NoMountingHoles"
 		(layer "B.Cu")
 		(at 192.5498 59.2777 180)
@@
 			)
 		)
-		(property "Footprint" "project:DIN41612_R_3x32_Male_Vertical_THT_Mirror"
+		(property "Footprint" "project:DIN41612_R_3x32_Male_Vertical_THT_Mirror_NoMountingHoles"
 			(at 0 -78.74 0)
 			(layer "B.Fab")
@@
 			(layer "B.Fab")
 		)
-		(fp_text user "c"
-			(at 4.49579 1.06033 0)
+		(fp_text user "a"
+			(at -0.58421 -80.772 0)
 			(unlocked yes)
 			(layer "B.SilkS")
@@
 			)
 		)
-		(fp_text user "a"
-			(at -0.58421 1.06033 0)
+		(fp_text user "1"
+			(at 1.9558 -81.153 0)
 			(unlocked yes)
 			(layer "B.SilkS")
@@
 			)
 		)
-		(fp_text user "1"
-			(at 1.9558 -81.153 0)
+		(fp_text user "c"
+			(at 4.49579 -80.772 0)
 			(unlocked yes)
 			(layer "B.SilkS")
@@
 		)
 		(fp_text user "a"
-			(at -0.58421 -80.772 0)
+			(at -0.58421 1.06033 0)
 			(unlocked yes)
 			(layer "B.SilkS")
@@
 		)
 		(fp_text user "c"
-			(at 4.49579 -80.772 0)
+			(at 4.49579 1.06033 0)
 			(unlocked yes)
 			(layer "B.SilkS")
