File: kicad/Performer-SE-PL-CL.kicad_sch (KiCad schematic)
At the start: 42 parts, among them IC1 MC68000P, J1 MAC_SE_PDS, U1 MC68030RC, U2 MC68881FN-SOC, U3 ATF16V8BJ, U4 ATF16V8BJ, U5 ATF16V8BJ, U6 ATF16V8BJ, U7 ATF16V8BJ

Commit message: Rename MC68030 Kicad footprint
Parts:
- U1: footprint Performer-SE-PL-CL:MPGA128 -> project:CPGA-169_MC68030
Changed lines of the file:
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@@
 			)
 		)
-		(property "Footprint" "Performer-SE-PL-CL:MPGA128"
+		(property "Footprint" "project:CPGA-169_MC68030"
 			(at 360.68 101.6 0)
 			(effects
@@
 			)
 		)
-		(property "Footprint" "Performer-SE-PL-CL:MPGA128"
+		(property "Footprint" "project:CPGA-169_MC68030"
 			(at 359.41 194.31 0)
 			(effects

Commit message: Update the MC68030 footprint
Parts:
- U1: footprint project:CPGA-169_MC68030 -> project:CPGA-128_Layout13x13_MC68030
Changed lines of the file:
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@@
 	(text "nc"
 		(exclude_from_sim no)
-		(at 304.8 55.88 0)
+		(at 279.4 55.88 0)
 		(effects
 			(font
@@
 			)
 		)
-		(property "Footprint" "project:CPGA-169_MC68030"
+		(property "Footprint" "project:CPGA-128_Layout13x13_MC68030"
 			(at 360.68 101.6 0)
 			(effects
@@
 			)
 		)
-		(property "Footprint" "project:CPGA-169_MC68030"
+		(property "Footprint" "project:CPGA-128_Layout13x13_MC68030"
 			(at 359.41 194.31 0)
 			(effects

Commit message: Update PDS footprint of the Performer-SE-PL-CL
Parts:
- J1: footprint project:DIN41612_R_3x32_Male_Vertical_THT_Mirror -> project:DIN41612_R_3x32_Male_Vertical_THT_Mirror_NoMountingHoles
Changed lines of the file:
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@@
 			)
 		)
-		(property "Footprint" "project:DIN41612_R_3x32_Male_Vertical_THT_Mirror"
+		(property "Footprint" "project:DIN41612_R_3x32_Male_Vertical_THT_Mirror_NoMountingHoles"
 			(at 53.34 106.68 0)
 			(effects
